File: nix_backplate/nix_backplate.kicad_pcb (KiCad board)
At the start: 2 copper layers, 100 x 30 mm, 0 parts

Commit message: Adjustments and text to backplate
Other:
- outline, holes or cut-outs redrawn
- board text added: "(7-15 VDC, 3 W)"
- board text added: "+"
- board text added: "-"
- board text added: "12 VDC"
- board text added: "JONAS ATTERTUN 2022"
- board text added: "OFF"
- board text added: "ON"
- board text added: "SET"
Changed lines of the file:
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@@
   (general
     (thickness 1.6)
-    (drawings 27)
+    (drawings 67)
     (tracks 0)
     (zones 0)
@@
     (uvia_drill 0.1)
   )
-  (gr_circle (center 185 115) (end 187.5 115) (layer Edge.Cuts) (width 0.15))
-  (gr_circle (center 165 115) (end 170.5 115) (layer F.SilkS) (width 0.15))
-  (gr_circle (center 145 115) (end 150.5 115) (layer F.SilkS) (width 0.15))
-  (gr_circle (center 129 115) (end 134.5 115) (layer F.SilkS) (width 0.15))
-  (gr_circle (center 113 115) (end 118.5 115) (layer F.SilkS) (width 0.15))
-  (gr_circle (center 195.5 104.5) (end 199 104.5) (layer F.SilkS) (width 0.15))
-  (gr_circle (center 195.5 125.5) (end 199 125.5) (layer F.SilkS) (width 0.15))
-  (gr_circle (center 104.5 125.5) (end 108 125.5) (layer F.SilkS) (width 0.15))
+  (gr_arc (start 104.5 104.5) (end 104.5 100) (angle -90) (layer Edge.Cuts) (width 0.15))
+  (gr_arc (start 104.5 125.5) (end 100 125.5) (angle -90) (layer Edge.Cuts) (width 0.15))
+  (gr_arc (start 195.5 125.5) (end 195.5 130) (angle -90) (layer Edge.Cuts) (width 0.15))
+  (gr_arc (start 195.5 104.5) (end 200 104.5) (angle -90) (layer Edge.Cuts) (width 0.15))
+  (gr_arc (start 195.5 104.5) (end 199 104.5) (angle -90) (layer F.Mask) (width 1))
+  (gr_arc (start 195.5 125.5) (end 195.5 129) (angle -90) (layer F.Mask) (width 1))
+  (gr_arc (start 104.5 125.5) (end 101 125.5) (angle -90) (layer F.Mask) (width 1))
+  (gr_arc (start 104.5 104.5) (end 104.5 101) (angle -90) (layer F.Mask) (width 1))
+  (gr_arc (start 195.5 104.5) (end 199 104.5) (angle -90) (layer F.Cu) (width 1))
+  (gr_arc (start 195.5 125.5) (end 195.5 129) (angle -90) (layer F.Cu) (width 1))
+  (gr_arc (start 104.5 125.5) (end 101 125.5) (angle -90) (layer F.Cu) (width 1))
+  (gr_arc (start 104.5 104.5) (end 104.5 101) (angle -90) (layer F.Cu) (width 1))
+  (gr_line (start 199 104.5) (end 199 125.5) (layer F.Mask) (width 1))
+  (gr_line (start 199 104.5) (end 199 125.5) (layer F.Cu) (width 1))
+  (gr_line (start 101 104.5) (end 101 125.5) (layer F.Mask) (width 1))
+  (gr_line (start 101 104.5) (end 101 125.5) (layer F.Cu) (width 1))
+  (gr_line (start 104.5 129) (end 195.5 129) (layer F.Cu) (width 1))
+  (gr_line (start 104.5 129) (end 195.5 129) (layer F.Mask) (width 1))
+  (gr_line (start 104.5 101) (end 195.5 101) (layer F.Mask) (width 1))
+  (gr_line (start 104.5 101) (end 195.5 101) (layer F.Cu) (width 1))
+  (gr_circle (center 185 115) (end 191 115) (layer F.Mask) (width 0.15))
+  (gr_circle (center 168 115) (end 173.5 115) (layer F.Mask) (width 0.15))
+  (gr_circle (center 145 115) (end 150.5 115) (layer F.Mask) (width 0.15))
+  (gr_circle (center 129 115) (end 134.5 115) (layer F.Mask) (width 0.15))
+  (gr_circle (center 113 115) (end 118.5 115) (layer F.Mask) (width 0.15))
+  (gr_text "JONAS ATTERTUN 2022" (at 122 127) (layer F.Mask)
+    (effects (font (size 1.5 1.5) (thickness 0.3) italic))
+  )
+  (gr_text "JONAS ATTERTUN 2022" (at 122 127) (layer F.Cu)
+    (effects (font (size 1.5 1.5) (thickness 0.3) italic))
+  )
+  (gr_text OFF (at 185 124) (layer F.Mask)
+    (effects (font (size 2 2) (thickness 0.4)))
+  )
+  (gr_text ON (at 185 107) (layer F.Mask)
+    (effects (font (size 2 2) (thickness 0.4)))
+  )
+  (gr_text "(7-15 VDC, 3 W)" (at 168 124) (layer F.Mask)
+    (effects (font (size 1 1) (thickness 0.2)))
+  )
+  (gr_text "12 VDC" (at 168 107) (layer F.Mask)
+    (effects (font (size 2 2) (thickness 0.4)))
+  )
+  (gr_text - (at 145 107) (layer F.Mask)
+    (effects (font (size 2 2) (thickness 0.4)))
+  )
+  (gr_text + (at 129 107) (layer F.Mask)
+    (effects (font (size 2 2) (thickness 0.4)))
+  )
+  (gr_text SET (at 113 107) (layer F.Mask)
+    (effects (font (size 2 2) (thickness 0.4)))
+  )
+  (gr_text "(7-15 VDC, 3 W)" (at 168 124) (layer F.Cu)
+    (effects (font (size 1 1) (thickness 0.2)))
+  )
+  (gr_text "12 VDC" (at 168 107) (layer F.Cu)
+    (effects (font (size 2 2) (thickness 0.4)))
+  )
+  (gr_text OFF (at 185 124) (layer F.Cu)
+    (effects (font (size 2 2) (thickness 0.4)))
+  )
+  (gr_text ON (at 185 107) (layer F.Cu)
+    (effects (font (size 2 2) (thickness 0.4)))
+  )
+  (gr_text - (at 145 107) (layer F.Cu)
+    (effects (font (size 2 2) (thickness 0.4)))
+  )
+  (gr_text + (at 129 107) (layer F.Cu)
+    (effects (font (size 2 2) (thickness 0.4)))
+  )
+  (gr_text SET (at 113 107) (layer F.Cu)
+    (effects (font (size 2 2) (thickness 0.4)))
+  )
+  (gr_line (start 181.5 121.5) (end 181.5 108.5) (layer Dwgs.User) (width 0.15))
+  (gr_line (start 181.5 121.5) (end 188.5 121.5) (layer Dwgs.User) (width 0.15))
+  (gr_line (start 188.5 108.5) (end 188.5 121.5) (layer Dwgs.User) (width 0.15))
+  (gr_line (start 181.5 108.5) (end 188.5 108.5) (layer Dwgs.User) (width 0.15))
+  (gr_circle (center 185 115) (end 188 115) (layer Edge.Cuts) (width 0.15))
+  (gr_circle (center 168 115) (end 173.5 115) (layer F.Cu) (width 0.15))
+  (gr_circle (center 145 115) (end 150.5 115) (layer F.Cu) (width 0.15))
+  (gr_circle (center 129 115) (end 134.5 115) (layer F.Cu) (width 0.15))
+  (gr_circle (center 113 115) (end 118.5 115) (layer F.Cu) (width 0.15))
+  (gr_circle (center 195.5 104.5) (end 199 104.5) (layer Dwgs.User) (width 0.15))
+  (gr_circle (center 195.5 125.5) (end 199 125.5) (layer Dwgs.User) (width 0.15))
+  (gr_circle (center 104.5 125.5) (end 108 125.5) (layer Dwgs.User) (width 0.15))
   (gr_circle (center 195.5 104.5) (end 197.25 104.5) (layer Edge.Cuts) (width 0.15))
   (gr_circle (center 195.5 125.5) (end 197.25 125.5) (layer Edge.Cuts) (width 0.15))
   (gr_circle (center 104.5 125.5) (end 106.25 125.5) (layer Edge.Cuts) (width 0.15))
-  (gr_arc (start 196.5 126.5) (end 196.5 130) (angle -90) (layer Edge.Cuts) (width 0.15))
-  (gr_arc (start 196.5 103.5) (end 200 103.5) (angle -90) (layer Edge.Cuts) (width 0.15))
-  (gr_arc (start 103.5 126.5) (end 100 126.5) (angle -90) (layer Edge.Cuts) (width 0.15))
-  (gr_arc (start 103.5 103.5) (end 103.5 100) (angle -90) (layer Edge.Cuts) (width 0.15))
-  (gr_circle (center 104.5 104.5) (end 108 104.5) (layer F.SilkS) (width 0.15))
+  (gr_circle (center 104.5 104.5) (end 108 104.5) (layer Dwgs.User) (width 0.15))
   (gr_circle (center 104.5 104.5) (end 106.25 104.5) (layer Edge.Cuts) (width 0.15))
-  (gr_circle (center 185 115) (end 193.5 115) (layer F.SilkS) (width 0.15))
-  (gr_circle (center 185 115) (end 191 115) (layer Edge.Cuts) (width 0.15))
-  (gr_circle (center 165 115) (end 169 115) (layer Edge.Cuts) (width 0.15))
+  (gr_circle (center 185 115) (end 191 115) (layer F.Cu) (width 0.15))
+  (gr_circle (center 168 115) (end 172 115) (layer Edge.Cuts) (width 0.15))
   (gr_circle (center 113 115) (end 116.5 115) (layer Edge.Cuts) (width 0.15))
   (gr_circle (center 145 115) (end 148.5 115) (layer Edge.Cuts) (width 0.15))
   (gr_circle (center 129 115) (end 132.5 115) (layer Edge.Cuts) (width 0.15))
-  (gr_line (start 100 103.5) (end 100 126.5) (layer Edge.Cuts) (width 0.15))
-  (gr_line (start 103.5 100) (end 196.5 100) (layer Edge.Cuts) (width 0.15))
-  (gr_line (start 200 103.5) (end 200 126.5) (layer Edge.Cuts) (width 0.15))
-  (gr_line (start 103.5 130) (end 196.5 130) (layer Edge.Cuts) (width 0.15))
+  (gr_line (start 100 104.5) (end 100 125.5) (layer Edge.Cuts) (width 0.15))
+  (gr_line (start 104.5 100) (end 195.5 100) (layer Edge.Cuts) (width 0.15))
+  (gr_line (start 200 104.5) (end 200 125.5) (layer Edge.Cuts) (width 0.15))
+  (gr_line (start 104.5 130) (end 195.5 130) (layer Edge.Cuts) (width 0.15))
 )
